Commit message: ack controller exception?

File: urdf/control.urdf.xacro (robot description, xacro)
@@ -6,4 +6,12 @@
       </hardware>
       <joint name="left_front_wheel_joint">
+          <command_interface name="position"/>
+          <state_interface name="position"/>
+      </joint>
+      <joint name="right_front_wheel_joint">
+          <command_interface name="position"/>
+          <state_interface name="position"/>
+      </joint>
+      <joint name="left_middle_wheel_joint">
           <command_interface name="velocity">
               <param name="min">-10</param>
@@ -11,7 +19,6 @@
           </command_interface>
           <state_interface name="velocity"/>
-          <state_interface name="position"/>
       </joint>
-      <joint name="right_front_wheel_joint">
+      <joint name="right_middle_wheel_joint">
           <command_interface name="velocity">
               <param name="min">-10</param>
@@ -19,4 +26,11 @@
           </command_interface>
           <state_interface name="velocity"/>
+      </joint>
+      <joint name="left_rear_wheel_joint">
+          <command_interface name="position"/>
+          <state_interface name="position"/>
+      </joint>
+      <joint name="right_rear_wheel_joint">
+          <command_interface name="position"/>
           <state_interface name="position"/>
       </joint>
