Commit message: fix position of link

File: urdf/eureka.urdf.xacro (robot description, xacro)
@@ -11,5 +11,5 @@
   <xacro:property name="wheel_mass" value="4.0"/>
   <xacro:property name="wheel_offset_x" value="0.4"/>
-  <xacro:property name="wheel_offset_y" value="0.3"/>
+  <xacro:property name="wheel_offset_y" value="0.4"/>
   <xacro:property name="wheel_offset_z" value="0.4"/>
   <material name="white">
@@ -24,16 +24,6 @@
   <link name="base_link">
   </link>
-  <joint name="base_footprint_joint" type="fixed">
-      <parent link="base_link"/>
-      <child link="base_footprint"/>
-      <origin xyz="0 0 0" rpy="0 0 0"/>
-  </joint>
   <link name="base_footprint">
   </link>
-  <joint name="chassis_joint" type="fixed">
-      <parent link="base_link"/>
-      <child link="chassis"/>
-      <origin xyz="0 0 ${wheel_offset_z}"/>
-  </joint>
   <link name="chassis">
     <visual>
@@ -54,13 +44,4 @@
     </xacro:inertial_box>
   </link>
-  <gazebo reference="chassis">
-      <material>Gazebo/Orange</material>
-  </gazebo>
-  <joint name="left_rear_wheel_joint" type="continuous">
-      <parent link="base_link"/>
-      <child link="left_rear_wheel"/>
-      <origin xyz="${-wheel_offset_x} ${wheel_offset_y} 0" rpy="-${pi/2} 0 0" />
-      <axis xyz="0 0 1"/>
-  </joint>
   <link name="left_rear_wheel">
     <visual>
@@ -79,7 +60,4 @@
     </xacro:inertial_cylinder>
   </link>
-  <gazebo reference="left_rear_wheel">
-      <material>Gazebo/Blue</material>
-  </gazebo>
   <link name="left_middle_wheel">
     <visual>
@@ -98,7 +76,4 @@
     </xacro:inertial_cylinder>
   </link>
-  <gazebo reference="left_middle_wheel">
-      <material>Gazebo/Blue</material>
-  </gazebo>
   <link name="left_front_wheel">
     <visual>
@@ -117,7 +92,4 @@
     </xacro:inertial_cylinder>
   </link>
-  <gazebo reference="left_front_wheel">
-      <material>Gazebo/Blue</material>
-  </gazebo>
   <link name="right_rear_wheel">
     <visual>
@@ -136,7 +108,4 @@
     </xacro:inertial_cylinder>
   </link>
-  <gazebo reference="right_rear_wheel">
-      <material>Gazebo/Blue</material>
-  </gazebo>
   <link name="right_middle_wheel">
     <visual>
@@ -155,7 +124,4 @@
     </xacro:inertial_cylinder>
   </link>
-  <gazebo reference="right_middle_wheel">
-      <material>Gazebo/Blue</material>
-  </gazebo>
   <link name="right_front_wheel">
     <visual>
@@ -174,7 +140,21 @@
     </xacro:inertial_cylinder>
   </link>
-  <gazebo reference="right_front_wheel">
-      <material>Gazebo/Blue</material>
-  </gazebo>
+  <xacro:include filename="$(find eureka_simulation)/urdf/gazebo_material.urdf.xacro"/>
+  <joint name="base_footprint_joint" type="fixed">
+      <parent link="base_link"/>
+      <child link="base_footprint"/>
+      <origin xyz="0 0 0" rpy="0 0 0"/>
+  </joint>
+  <joint name="chassis_joint" type="fixed">
+      <parent link="base_link"/>
+      <child link="chassis"/>
+      <origin xyz="${-chassis_length/2} 0 0"/>
+  </joint>
+  <joint name="left_rear_wheel_joint" type="continuous">
+      <parent link="base_link"/>
+      <child link="left_rear_wheel"/>
+      <origin xyz="${-wheel_offset_x} ${wheel_offset_y} 0" rpy="-${pi/2} 0 0" />
+      <axis xyz="0 0 1"/>
+  </joint>
   <joint name="left_middle_wheel_joint" type="continuous">
       <parent link="base_link"/>

Commit message: fix axis in urdf

File: urdf/eureka.urdf.xacro (robot description, xacro)
@@ -23,6 +23,4 @@
   </material>
   <link name="base_link">
-  </link>
-  <link name="base_footprint">
   </link>
   <link name="chassis">
@@ -141,9 +139,4 @@
   </link>
   <xacro:include filename="$(find eureka_simulation)/urdf/gazebo_material.urdf.xacro"/>
-  <joint name="base_footprint_joint" type="fixed">
-      <parent link="base_link"/>
-      <child link="base_footprint"/>
-      <origin xyz="0 0 0" rpy="0 0 0"/>
-  </joint>
   <joint name="chassis_joint" type="fixed">
       <parent link="base_link"/>
@@ -173,5 +166,5 @@
       <child link="right_rear_wheel"/>
       <origin xyz="${-wheel_offset_x} ${-wheel_offset_y} 0" rpy="-${pi/2} 0 0" />
-      <axis xyz="0 0 -1"/>
+      <axis xyz="0 0 1"/>
   </joint>
   <joint name="right_middle_wheel_joint" type="continuous">
@@ -179,5 +172,5 @@
       <child link="right_middle_wheel"/>
       <origin xyz="0 ${-wheel_offset_y} 0" rpy="-${pi/2} 0 0" />
-      <axis xyz="0 0 -1"/>
+      <axis xyz="0 0 1"/>
   </joint>
   <joint name="right_front_wheel_joint" type="continuous">
@@ -185,5 +178,5 @@
       <child link="right_front_wheel"/>
       <origin xyz="${wheel_offset_x} ${-wheel_offset_y} 0" rpy="-${pi/2} 0 0" />
-      <axis xyz="0 0 -1"/>
+      <axis xyz="0 0 1"/>
   </joint>
   <xacro:include filename="control.urdf.xacro"/>

Commit message: wrong rocky-bogie chassis

File: urdf/eureka.urdf.xacro (robot description, xacro)
@@ -147,5 +147,5 @@
       <parent link="base_link"/>
       <child link="left_rear_wheel"/>
-      <origin xyz="${-wheel_offset_x} ${wheel_offset_y} 0" rpy="-${pi/2} 0 0" />
+      <origin xyz="${-wheel_offset_x} ${wheel_offset_y} 0.02" rpy="-${pi/2} 0 0" />
       <axis xyz="0 0 1"/>
   </joint>
@@ -165,5 +165,5 @@
       <parent link="base_link"/>
       <child link="right_rear_wheel"/>
-      <origin xyz="${-wheel_offset_x} ${-wheel_offset_y} 0" rpy="-${pi/2} 0 0" />
+      <origin xyz="${-wheel_offset_x} ${-wheel_offset_y} 0.02" rpy="-${pi/2} 0 0" />
       <axis xyz="0 0 1"/>
   </joint>

Commit message: add laser sensor

File: urdf/eureka.urdf.xacro (robot description, xacro)
@@ -2,5 +2,4 @@
 <robot xmlns:xacro="http://www.ros.org/wiki/xacro" name="eureka">
   <xacro:include filename="$(find eureka_simulation)/urdf/inertial_macros.xacro"/>
-  <!-- <xacro:include filename="$(find eureka_simulation)/urdf/eureka_control.urdf.xacro"/> -->
   <xacro:property name="chassis_length" value="0.76"/>
   <xacro:property name="chassis_width" value="0.5"/>
@@ -13,13 +12,5 @@
   <xacro:property name="wheel_offset_y" value="0.4"/>
   <xacro:property name="wheel_offset_z" value="0.4"/>
-  <material name="white">
-      <color rgba="1 1 1 1" />
-  </material>
-  <material name="orange">
-      <color rgba="1 0.3 0.1 1"/>
-  </material>
-  <material name="blue">
-      <color rgba="0.2 0.2 1 1"/>
-  </material>
+  <xacro:include filename="materials.urdf.xacro"/>
   <link name="base_link">
   </link>
@@ -180,5 +171,6 @@
       <axis xyz="0 0 1"/>
   </joint>
+  <xacro:include filename="sensor.urdf.xacro"/>
   <xacro:include filename="control.urdf.xacro"/>
-  <xacro:include filename="materials.urdf.xacro"/>
+  <xacro:include filename="gazebo_material.urdf.xacro"/>
 </robot>

File: urdf/materials.urdf.xacro (robot description, xacro)
@@ -4,3 +4,15 @@
     <color rgba="0.700 0.700 0.700 1.000"/>
   </material>
+  <material name="white">
+      <color rgba="1 1 1 1" />
+  </material>
+  <material name="orange">
+      <color rgba="1 0.3 0.1 1"/>
+  </material>
+  <material name="blue">
+      <color rgba="0.2 0.2 1 1"/>
+  </material>
+  <material name="black">
+      <color rgba="0 0 0 1"/>
+  </material>
 </robot>

Commit message: tune controllers parametrs to fine odometry and add new world.

File: urdf/eureka.urdf.xacro (robot description, xacro)
@@ -2,5 +2,5 @@
 <robot xmlns:xacro="http://www.ros.org/wiki/xacro" name="eureka">
   <xacro:include filename="$(find eureka_simulation)/urdf/inertial_macros.xacro"/>
-  <xacro:property name="chassis_length" value="0.76"/>
+  <xacro:property name="chassis_length" value="0.8"/>
   <xacro:property name="chassis_width" value="0.5"/>
   <xacro:property name="chassis_height" value="0.3"/>

Commit message: add new world and depth camera

File: urdf/eureka.urdf.xacro (robot description, xacro)
@@ -10,5 +10,5 @@
   <xacro:property name="wheel_mass" value="4.0"/>
   <xacro:property name="wheel_offset_x" value="0.4"/>
-  <xacro:property name="wheel_offset_y" value="0.4"/>
+  <xacro:property name="wheel_offset_y" value="0.5"/>
   <xacro:property name="wheel_offset_z" value="0.4"/>
   <xacro:include filename="materials.urdf.xacro"/>
@@ -138,11 +138,11 @@
       <parent link="base_link"/>
       <child link="left_rear_wheel"/>
-      <origin xyz="${-wheel_offset_x} ${wheel_offset_y} 0.02" rpy="-${pi/2} 0 0" />
-      <axis xyz="0 0 1"/>
+      <origin xyz="${-wheel_offset_x} ${wheel_offset_y} 0" rpy="-${pi/2} 0 0" />
+      <axis xyz="0 -1 1"/>
   </joint>
   <joint name="left_middle_wheel_joint" type="continuous">
       <parent link="base_link"/>
       <child link="left_middle_wheel"/>
-      <origin xyz="0 ${wheel_offset_y} 0" rpy="-${pi/2} 0 0" />
+      <origin xyz="0 ${wheel_offset_y} -0.001" rpy="-${pi/2} 0 0" />
       <axis xyz="0 0 1"/>
   </joint>
@@ -151,16 +151,16 @@
       <child link="left_front_wheel"/>
       <origin xyz="${wheel_offset_x} ${wheel_offset_y} 0" rpy="-${pi/2} 0 0" />
-      <axis xyz="0 0 1"/>
+      <axis xyz="0 -1 1"/>
   </joint>
   <joint name="right_rear_wheel_joint" type="continuous">
       <parent link="base_link"/>
       <child link="right_rear_wheel"/>
-      <origin xyz="${-wheel_offset_x} ${-wheel_offset_y} 0.02" rpy="-${pi/2} 0 0" />
-      <axis xyz="0 0 1"/>
+      <origin xyz="${-wheel_offset_x} ${-wheel_offset_y} 0" rpy="-${pi/2} 0 0" />
+      <axis xyz="0 -1 1"/>
   </joint>
   <joint name="right_middle_wheel_joint" type="continuous">
       <parent link="base_link"/>
       <child link="right_middle_wheel"/>
-      <origin xyz="0 ${-wheel_offset_y} 0" rpy="-${pi/2} 0 0" />
+      <origin xyz="0 ${-wheel_offset_y} -0.001" rpy="-${pi/2} 0 0" />
       <axis xyz="0 0 1"/>
   </joint>
@@ -169,5 +169,5 @@
       <child link="right_front_wheel"/>
       <origin xyz="${wheel_offset_x} ${-wheel_offset_y} 0" rpy="-${pi/2} 0 0" />
-      <axis xyz="0 0 1"/>
+      <axis xyz="0 -1 1"/>
   </joint>
   <xacro:include filename="sensor.urdf.xacro"/>

File: urdf/sensor.urdf.xacro (robot description, xacro)
@@ -1,13 +1,8 @@
 <?xml version="1.0" ?>
 <robot xmlns:xacro="http://www.ros.org/wiki/xacro" >
-    <joint name="laser_joint" type="fixed">
-        <parent link="chassis"/>
-        <child link="laser_frame"/>
-        <origin xyz="${chassis_length/2} 0 ${chassis_height + 0.1}" rpy="0 0 0"/>
-    </joint>
-    <link name="laser_frame">
+    <link name="camera_link">
         <visual>
             <geometry>
-                <cylinder radius="0.05" length="0.04"/>
+                <box size="0.010 0.03 0.03"/>
             </geometry>
             <material name="black"/>
@@ -16,42 +11,42 @@
             <origin xyz="0 0 -0.05"/>
             <geometry>
-                <cylinder radius="0.01" length="0.1"/>
+                <cylinder radius="0.002" length="0.1"/>
             </geometry>
             <material name="black"/>
         </visual>
-        <collision>
-            <geometry>
-                <cylinder radius="0.05" length="0.04"/>
-            </geometry>
-        </collision>
-        <xacro:inertial_cylinder mass="0.1" length="0.04" radius="0.05">
-            <origin xyz="0 0 0" rpy="0 0 0"/>
-        </xacro:inertial_cylinder>
     </link>
-    <gazebo reference="laser_frame">
-        <material>Gazebo/Black</material>
-        <sensor name="laser" type="ray">
+    <link name="camera_link_optical"></link>
+    <joint name="camera_joint" type="fixed">
+        <parent link="chassis"/>
+        <child link="camera_link"/>
+        <origin xyz="${chassis_length} 0 ${chassis_height}" rpy="0 0.18 0"/>
+    </joint>
+    <joint name="camera_optical_joint" type="fixed">
+        <parent link="camera_link"/>
+        <child link="camera_link_optical"/>
+        <origin xyz="0 0 0" rpy="${-pi/2} 0 ${-pi/2}"/>
+    </joint>
+    <gazebo reference="camera_link">
+        <material>Gazebo/Red</material>
+        <sensor name="camera" type="depth">
             <pose> 0 0 0 0 0 0 </pose>
-            <visualize>false</visualize>
+            <visualize>true</visualize>
             <update_rate>10</update_rate>
-            <ray>
-                <scan>
-                    <horizontal>
-                        <samples>360</samples>
-                        <min_angle>-3.14</min_angle>
-                        <max_angle>3.14</max_angle>
-                    </horizontal>
-                </scan>
-                <range>
-                    <min>0.3</min>
-                    <max>12</max>
-                </range>
-            </ray>
-            <plugin name="laser_controller" filename="libgazebo_ros_ray_sensor.so">
-                <ros>
-                    <argument>~/out:=scan</argument>
-                </ros>
-                <output_type>sensor_msgs/LaserScan</output_type>
-                <frame_name>laser_frame</frame_name>
+            <camera>
+                <horizontal_fov>1.089</horizontal_fov>
+                <image>
+                    <format>B8G8R8</format>
+                    <width>640</width>
+                    <height>480</height>
+                </image>
+                <clip>
+                    <near>0.05</near>
+                    <far>8.0</far>
+                </clip>
+            </camera>
+            <plugin name="camera_controller" filename="libgazebo_ros_camera.so">
+                <frame_name>camera_link_optical</frame_name>
+                <min_depth>0.1</min_depth>
+                <max_depth>100.0</max_depth>
             </plugin>
         </sensor>
