Commit message: feat: add gps

File: description/eureka.urdf.xacro (robot description, xacro)
@@ -135,4 +135,8 @@
         <!-- <origin xyz="0.212 0 0.065" rpy="0 0 0"/> -->
     </xacro:sensor_asus_xtion>
+    <xacro:sensor_gps prefix="gps" parent="base_link">
+        <origin xyz="0 0 0" rpy="0 0 0"/>
+        <!-- <origin xyz="0.212 0 0.065" rpy="0 0 0"/> -->
+    </xacro:sensor_gps>
     <!-- wheels -->
     <xacro:corner_link lon_label="front" lat_label="left" reflect="1"/>

Commit message: feat: add new link + configure ekf

File: description/eureka.urdf.xacro (robot description, xacro)
@@ -102,4 +102,13 @@
     </ros2_control>
     <!-- The base link -->
+    <link name="base_footprint">
+        <visual>
+            <origin rpy="0 0 0" xyz="0 0 0" />
+            <geometry>
+                <box size="0.01 0.01 0.01"/>
+            </geometry>
+            <material name="orange" />
+        </visual>
+    </link>
     <link name="base_link">
         <visual>
@@ -111,4 +120,9 @@
         </visual>
     </link>
+    <joint name="truth_joint" type="fixed">
+        <origin rpy="0 0 0" xyz="0 0 0.205"/>
+        <parent link="base_footprint" />
+        <child link="base_link" />
+    </joint>
     <gazebo reference="base_link">
         <material>Gazebo/Orange</material>

Commit message: feat: move imu into the camera

File: description/eureka.urdf.xacro (robot description, xacro)
@@ -141,12 +141,12 @@
         <origin xyz="0.17 0 0.005" rpy="0 0 0"/>
     </xacro:sensor_hokuyo>
-    <xacro:sensor_imu prefix="imu" parent="base_link">
-        <!-- <origin xyz="-0.32 0 0.05" rpy="0 0.5 0"/> -->
-        <origin xyz="0 0 -0.04" rpy="0 0 0"/>
-    </xacro:sensor_imu>
     <xacro:sensor_asus_xtion prefix="camera" parent="base_link">
         <origin xyz="0.215 0 0.065" rpy="0 0.4 0"/>
         <!-- <origin xyz="0.212 0 0.065" rpy="0 0 0"/> -->
     </xacro:sensor_asus_xtion>
+    <xacro:sensor_imu prefix="imu" parent="camera_link">
+        <!-- <origin xyz="-0.32 0 0.05" rpy="0 0.5 0"/> -->
+        <origin xyz="0 0 0" rpy="0 0 0"/>
+    </xacro:sensor_imu>
     <xacro:sensor_gps prefix="gps" parent="base_link">
         <origin xyz="0 0 0" rpy="0 0 0"/>

Commit message: fix: clenup pakcage - divide launch by purpose - add eagleye pose estimator launch setup - add ORB SLAM vocabulary - fix mars2.world by deleting unused erueka model inside .world - add track voc.txt via git lfs - full independence from other eureka package

File: description/eureka.urdf.xacro (robot description, xacro)
@@ -15,5 +15,5 @@
     <gazebo>
         <plugin filename="libgazebo_ros2_control.so" name="gazebo_ros2_control">
-            <parameters>$(find eureka_simulation)/config/my_controllers.yaml</parameters>
+            <parameters>$(find eureka_simulation)/config/controller/my_controllers.yaml</parameters>
         </plugin>
     </gazebo>
@@ -143,5 +143,4 @@
     <xacro:sensor_asus_xtion prefix="camera" parent="base_link">
         <origin xyz="0.215 0 0.065" rpy="0 0.4 0"/>
-        <!-- <origin xyz="0.212 0 0.065" rpy="0 0 0"/> -->
     </xacro:sensor_asus_xtion>
     <xacro:sensor_imu prefix="imu" parent="camera_link">

File: description/sensors/all_sensors.urdf.xacro (robot description, xacro)
@@ -24,4 +24,6 @@
   <!-- Xtion -->
   <xacro:include filename="$(find eureka_simulation)/description/sensors/asus_xtion.urdf.xacro" />
+  <!-- Realsense d415 -->
+  <xacro:include filename="$(find eureka_simulation)/description/sensors/realsense_d415.urdf.xacro" />
   <!-- GPS -->
   <xacro:include filename="$(find eureka_simulation)/description/sensors/gps.urdf.xacro" />

File: description/sensors/asus_xtion.urdf.xacro (robot description, xacro)
@@ -73,14 +73,7 @@
           </image>
           <clip>
-            <near>0.3</near>
-            <far>8.0</far>
+            <near>0.01</near>
+            <far>50.0</far>
           </clip>
-	        <distortion>
-            <k1>0.00000001</k1>
-            <k2>0.00000001</k2>
-            <k3>0.00000001</k3>
-            <p1>0.00000001</p1>
-            <p2>0.00000001</p2>
-          </distortion>
         </camera>
         <plugin name="depth_camera_controller" filename="libgazebo_ros_camera.so">
@@ -145,6 +138,6 @@
           </ros>
           <frame_name>camera_frame</frame_name>
-          <min_depth>0.3</min_depth>
-          <max_depth>8.0</max_depth>
+          <min_depth>0.01</min_depth>
+          <max_depth>100.0</max_depth>
         </plugin>
       </sensor>

Commit message: fix: configure yaml's - remove z axis in position from odom_rgbd and infantate z coord - correct foorprint in yaml - g2o from orb can't process optimization in rtabmap, so swap it to TORO - little correct rotate camera -  set new logging policy for launche's

File: description/eureka.urdf.xacro (robot description, xacro)
@@ -142,5 +142,5 @@
     </xacro:sensor_hokuyo>
     <xacro:sensor_asus_xtion prefix="camera" parent="base_link">
-        <origin xyz="0.215 0 0.065" rpy="0 0.4 0"/>
+        <origin xyz="0.215 0 0.065" rpy="0 0.3 0"/>
     </xacro:sensor_asus_xtion>
     <xacro:sensor_imu prefix="imu" parent="camera_link">
